Commit message: Added latest models

File: urdf/doorHinge_inf.urdf (robot description, URDF)
Before this commit: robot clutch_container, 1 links, 0 joints
Links:
- removed link clutch_container
- added link doorHinge, mass 1.0; collision mesh filename=../meshes/PSA/doorHinge_inf.obj scale=1 1 1; visual mesh filename=../meshes/PSA/doorHinge_inf.obj scale=1 1 1

File: urdf/doorHinge_sup.urdf (robot description, URDF)
Before this commit: robot tableDining, 1 links, 0 joints
Links:
- removed link tableDining
- added link doorHinge, mass 1.0; collision mesh filename=../meshes/PSA/doorHinge_sup.obj scale=1 1 1; visual mesh filename=../meshes/PSA/doorHinge_sup.obj scale=1 1 1

File: urdf/wheelPivot_right.urdf (robot description, URDF)
Before this commit: robot clutch, 1 links, 0 joints
Links:
- removed link clutch
- added link wheelPivot, mass 2.5; collision mesh filename=../meshes/PSA/wheelPivot_right.obj scale=1 1 1; visual mesh filename=../meshes/PSA/wheelPivot_right.obj scale=1 1 1
