Commit message: Added scene files

File: urdf/wheelPivot_left.urdf (robot description, URDF)
Before this commit: robot wheelPivot_left, 1 links, 0 joints
Links:
- link wheelPivot: geometry collision mesh filename=../meshes/PSA/wheelPivot_left.blend scale=1 1 1; visual mesh filename=../meshes/PSA/wheelPivot_left.blend scale=1 1 1

Commit message: Added models

File: urdf/wheelPivot_left.urdf (robot description, URDF)
Before this commit: robot wheelPivot_left, 1 links, 0 joints
Links:
- link wheelPivot: geometry collision mesh filename=../meshes/PSA/wheelPivot_left.dae scale=1 1 1; visual mesh filename=../meshes/PSA/wheelPivot_left.dae scale=1 1 1
