Commit message: Added scenes from Friday

File: urdf/Rubber_obturator.urdf (robot description, URDF)
Before this commit: robot rubber, 1 links, 0 joints
Links:
- link rubber: geometry collision mesh filename=../meshes/PSA/Rubber_obturator.dae scale=1 1 1; visual mesh filename=../meshes/PSA/Rubber_obturator.dae scale=1 1 1

File: urdf/clutch.urdf (robot description, URDF)
Before this commit: robot clutch, 1 links, 0 joints
Links:
- link clutch: geometry collision mesh filename=../meshes/PSA/clutchSensor.dae scale=1 1 1; visual mesh filename=../meshes/PSA/clutchSensor.dae scale=1 1 1

File: urdf/robots/sdh.urdf (robot description, URDF)
Before this commit: robot sdh, 13 links, 12 joints
Links:
- link finger_11_link: geometry collision mesh filename=../../meshes/sdh/knuckle.dae; visual mesh filename=../../meshes/sdh/knuckle.dae
- link finger_12_link: geometry collision mesh filename=../../meshes/sdh/finger.dae; visual mesh filename=../../meshes/sdh/finger.dae
- link finger_13_link: geometry collision mesh filename=../../meshes/sdh/finger_tip.dae; visual mesh filename=../../meshes/sdh/finger_tip.dae
- link finger_21_link: geometry collision mesh filename=../../meshes/sdh/knuckle.dae; visual mesh filename=../../meshes/sdh/knuckle.dae
- link finger_22_link: geometry collision mesh filename=../../meshes/sdh/finger.dae; visual mesh filename=../../meshes/sdh/finger.dae
- link finger_23_link: geometry collision mesh filename=../../meshes/sdh/finger_tip.dae; visual mesh filename=../../meshes/sdh/finger_tip.dae
- link palm_link: geometry collision mesh filename=../../meshes/sdh/palm.dae; visual mesh filename=../../meshes/sdh/palm.dae
- link thumb_1_link: geometry collision mesh filename=../../meshes/sdh/knuckle.dae; visual mesh filename=../../meshes/sdh/knuckle.dae
- link thumb_2_link: geometry collision mesh filename=../../meshes/sdh/finger.dae; visual mesh filename=../../meshes/sdh/finger.dae
- link thumb_3_link: geometry collision mesh filename=../../meshes/sdh/finger_tip.dae; visual mesh filename=../../meshes/sdh/finger_tip.dae
Joints:
- joint palm_joint: type floating -> fixed

File: urdf/wheelPivot_right.urdf (robot description, URDF)
Before this commit: robot wheelPivot_right, 1 links, 0 joints
Links:
- link wheelPivot: geometry collision mesh filename=../meshes/PSA/wheelPivot_right.dae scale=1 1 1; visual mesh filename=../meshes/PSA/wheelPivot_right.dae scale=1 1 1
