Commit message: Added new desk and erased old escritorio4

File: urdf/graspTests/simpleDesk.urdf (robot description, URDF)
Before this commit: robot escritorio4, 1 links, 0 joints
Links:
- removed link escritorio4
- added link simpleDesk, mass 0.5; collision mesh filename=../../meshes/dae/graspTests/simpleDesk.dae scale=1 1 1; visual mesh filename=../../meshes/dae/graspTests/simpleDesk.dae scale=1 1 1
