Commit message: Added scenes

File: urdf/graspTests/wineBottle_1.urdf (robot description, URDF)
Before this commit: robot wineBouteille_1, 1 links, 0 joints
Links:
- link wineBouteille_1: geometry collision mesh filename=../../meshes/dae/graspTests/wineBouteille_centered.dae scale=1 1 1; visual mesh filename=../../meshes/dae/graspTests/wineBouteille_centered.dae scale=1 1 1
