Commit message: Added crap

File: urdf/robots/bhand_old.urdf (robot description, URDF)
Before this commit: robot bhand_model, 9 links, 8 joints
Joints:
- joint finger_1_dist_joint: axis 0 0 -1 -> 0 0 1; limit lower=0 upper=0.785 effort=0 velocity=0 -> lower=-0.785 upper=0 effort=0 velocity=0
- joint finger_1_med_joint: axis 0 0 -1 -> 0 0 1; limit lower=0 upper=2.44 effort=0 velocity=0 -> lower=-2.44 upper=0 effort=0 velocity=0
- joint finger_2_dist_joint: axis 0 0 -1 -> 0 0 1; limit lower=0 upper=0.785 effort=0 velocity=0 -> lower=-0.785 upper=0 effort=0 velocity=0
- joint finger_2_med_joint: axis 0 0 -1 -> 0 0 1; limit lower=0 upper=2.44 effort=0 velocity=0 -> lower=-2.44 upper=0 effort=0 velocity=0
- joint finger_3_dist_joint: axis 0 0 -1 -> 0 0 1; limit lower=0 upper=0.785 effort=0 velocity=0 -> lower=-0.785 upper=0 effort=0 velocity=0
- joint finger_3_med_joint: axis 0 0 -1 -> 0 0 1; limit lower=0 upper=2.44 effort=0 velocity=0 -> lower=-2.44 upper=0 effort=0 velocity=0

File: urdf/robots/iri_wam_testNoFixed.urdf (robot description, URDF)
Before this commit: robot wam_model, 10 links, 9 joints
Links:
- removed link forearm_link
Joints:
- removed joint elbow_fixed_joint
- joint wrist_yaw_joint: origin xyz=0 0 0.1993 rpy=0 0 0 -> xyz=-0.045 -0.1263 0 rpy=-1.57 0 3.1416; parent forearm_link -> elbow_link
