Commit message: Added changes of Sunday

File: urdf/robots/iri_wam.urdf (robot description, URDF)
Before this commit: robot wam_model, 10 links, 9 joints
Links:
- removed link forearm_link
Joints:
- removed joint elbow_fixed_joint
- joint wrist_yaw_joint: origin xyz=0 0 0.1993 rpy=0 0 0 -> xyz=-0.045 -0.1263 0 rpy=-1.5708 0 3.1416; parent forearm_link -> elbow_link
