Commit message: Added stuff

File: urdf/rssModels/blueCup_sketchup.urdf (robot description, URDF)
Before this commit: robot wineBouteille_1, 1 links, 0 joints
Links:
- removed link wineBouteille_1
- added link blueCup, mass 0.5; collision mesh filename=../../meshes/rssModels/blueCup_sketchup.dae scale=1 1 1; visual mesh filename=../../meshes/rssModels/blueCup_sketchup.dae scale=1 1 1

File: urdf/rssModels/tetrapak_sketchup.urdf (robot description, URDF)
Before this commit: robot wineBouteille_1, 1 links, 0 joints
Links:
- removed link wineBouteille_1
- added link tetrapak, mass 0.5; collision mesh filename=../../meshes/rssModels/tetrapak_sketchup.dae scale=1 1 1; visual mesh filename=../../meshes/rssModels/tetrapak_sketchup.dae scale=1 1 1
