Commit message: Added left and right also for LWA4

File: robots/hubo/urdf/huboLeftArm.urdf (robot description, URDF)
Before this commit: robot leftArm, 9 links, 8 joints
Joints:
- joint L0_joint: type fixed -> floating

File: robots/hubo/urdf/huboRightArm.urdf (robot description, URDF)
Before this commit: robot huboRightArm, 9 links, 8 joints
Joints:
- joint L0_joint: type fixed -> floating
