Commit message: Added slight changes

File: robots/hubo/urdf/huboLeftHand.urdf (robot description, URDF)
Before this commit: robot leftHand, 11 links, 10 joints
Joints:
- joint LF12: limit lower=-1.5 upper=.1 effort=10.0 velocity=2.0 -> lower=0.1 upper=1.5 effort=10.0 velocity=2.0
- joint LF13: limit lower=-1.5 upper=.1 effort=10.0 velocity=2.0 -> lower=0.1 upper=1.5 effort=10.0 velocity=2.0
- joint LF22: limit lower=-1.5 upper=.1 effort=10.0 velocity=2.0 -> lower=0.1 upper=1.5 effort=10.0 velocity=2.0
- joint LF23: limit lower=-1.5 upper=.1 effort=10.0 velocity=2.0 -> lower=0.1 upper=1.5 effort=10.0 velocity=2.0
- joint LF31: axis 0 -1 0 -> 0 1 0
- joint LF32: axis (none) -> 0 1 0; limit lower=-1.5 upper=.1 effort=10.0 velocity=2.0 -> lower=-0.1 upper=1.5 effort=10.0 velocity=2.0
- joint LF33: axis 0 -1 0 -> 0 1 0; limit lower=-1.5 upper=.1 effort=10.0 velocity=2.0 -> lower=-0.1 upper=1.5 effort=10.0 velocity=2.0
