Commit message: Fixed hubo right hand limits and change name to root link of LWA4 mid

File: robots/hubo/urdf/huboRightHand.urdf (robot description, URDF)
Before this commit: robot huboRightHand, 14 links, 13 joints
Joints:
- joint RF12: limit lower=-1.5 upper=.1 effort=10.0 velocity=2.0 -> lower=0.1 upper=1.5 effort=10.0 velocity=2.0
- joint RF13: limit lower=-1.5 upper=.1 effort=10.0 velocity=2.0 -> lower=0.1 upper=1.5 effort=10.0 velocity=2.0
- joint RF22: limit lower=-1.5 upper=.1 effort=10.0 velocity=2.0 -> lower=0.1 upper=1.5 effort=10.0 velocity=2.0
- joint RF23: limit lower=-1.5 upper=.1 effort=10.0 velocity=2.0 -> lower=0.1 upper=1.5 effort=10.0 velocity=2.0
- joint RF31: axis 0 -1 0 -> 0 1 0
- joint RF32: axis 0 -1 0 -> 0 1 0; limit lower=-1.5 upper=.1 effort=10.0 velocity=2.0 -> lower=-0.1 upper=1.5 effort=10.0 velocity=2.0
- joint RF33: axis 0 -1 0 -> 0 1 0; limit lower=-1.5 upper=.1 effort=10.0 velocity=2.0 -> lower=-0.1 upper=1.5 effort=10.0 velocity=2.0
- joint RF41: axis 0 -1 0 -> 0 1 0
- joint RF42: axis 0 -1 0 -> 0 1 0; limit lower=-1.5 upper=.1 effort=10.0 velocity=2.0 -> lower=-0.1 upper=1.5 effort=10.0 velocity=2.0
- joint RF43: axis 0 -1 0 -> 0 1 0; limit lower=-1.5 upper=.1 effort=10.0 velocity=2.0 -> lower=-0.1 upper=1.5 effort=10.0 velocity=2.0
