Commit message: Added bimanual scenario

File: robots/lwa4d/urdf/lwa4d_left.urdf (robot description, URDF)
Before this commit: robot lwa4d, 9 links, 8 joints
Links:
- link L0_link: geometry 

File: robots/lwa4d/urdf/lwa4d_right.urdf (robot description, URDF)
Before this commit: robot lwa4d, 9 links, 8 joints
Links:
- link L0_link: geometry 
