Commit message: Added physical models + table with marker

File: robots/lwa4d/urdf/lwa4d_left_phys.urdf (robot description, URDF)
Before this commit: robot lwa4d, 9 links, 8 joints
Links:
- link L5_link: geometry collision mesh filename=../meshes/arm_5_link_phys.dae; visual mesh filename=../meshes/arm_5_link_phys.dae
Joints:
- joint L1_joint: origin xyz=0 -0.1375 0 rpy=-1.5708 3.1416 0 -> xyz=0 0.12 0 rpy=1.57 3.1416 0
- joint L2_joint: axis 0 0 1 -> 0 0 -1
- joint L4_joint: axis 0 0 1 -> 0 0 -1
- joint L6_joint: axis 0 0 1 -> 0 0 -1
- joint L7_joint: axis 0 0 1 -> 0 0 -1

File: robots/lwa4d/urdf/lwa4d_right_phys.urdf (robot description, URDF)
Before this commit: robot lwa4d, 9 links, 8 joints
Links:
- link L5_link: geometry collision mesh filename=../meshes/arm_5_link_phys.dae; visual mesh filename=../meshes/arm_5_link_phys.dae
Joints:
- joint L1_joint: origin xyz=0 -0.1375 0 rpy=-1.5708 3.1416 0 -> xyz=0 0.12 0 rpy=1.57 3.1416 0
- joint L2_joint: axis 0 0 1 -> 0 0 -1
- joint L4_joint: axis 0 0 1 -> 0 0 -1
- joint L6_joint: axis 0 0 1 -> 0 0 -1
- joint L7_joint: axis 0 0 1 -> 0 0 -1
