Commit message: Added F/T in urdf and meshes. Cleaned up a bit the lwa4d folder

File: robots/lwa4d/urdf/lwa4d_right_phys.urdf (robot description, URDF)
Before this commit: robot lwa4d_right, 9 links, 8 joints
Links:
- link L7_link: geometry collision mesh filename=../meshes/arm_7_FT_tool_changers_link.dae; visual mesh filename=../meshes/arm_7_FT_tool_changers_link.dae
Joints:
- joint L7_joint: origin xyz=0 -0.075 0 rpy=-1.57 0 0 -> xyz=0 -0.1672 0 rpy=-1.57 0 0

Commit message: Corrected limits for joint 1 and a couple more according to the data sheet. Values used to be 2PI instead of PI

File: robots/lwa4d/urdf/lwa4d_right_phys.urdf (robot description, URDF)
Before this commit: robot lwa4d_right, 9 links, 8 joints
Joints:
- joint L1_joint: limit lower=-6.2831853 upper=6.2831853 effort=370 velocity=2.0 -> lower=-3.14157 upper=3.14157 effort=370 velocity=2.0
- joint L3_joint: limit lower=-6.2831853 upper=6.2831853 effort=176 velocity=2.0 -> lower=-3.14157 upper=3.14157 effort=176 velocity=2.0
- joint L5_joint: limit lower=-6.2831853 upper=6.2831853 effort=41.6 velocity=2.0 -> lower=-3.14157 upper=3.14157 effort=41.6 velocity=2.0
- joint L7_joint: limit lower=-6.2831853 upper=6.2831853 effort=9.6 velocity=2.0 -> lower=-3.14157 upper=3.14157 effort=9.6 velocity=2.0
