Commit message: Added grasPrim

File: objects/tetrapak/urdf/tetrapak.urdf (robot description, URDF)
Before this commit: robot tetrapak, 1 links, 0 joints
Links:
- link tetrapak: geometry collision mesh filename=../meshes/tetrapak.dae scale=1 1 1; visual mesh filename=../meshes/tetrapak.dae scale=1 1 1
