Commit message: Added hand

File: robots/alita/urdf/alita_left.urdf (robot description, URDF)
Before this commit: robot alita_left, 11 links, 10 joints
Links:
- removed link lFingerA
- removed link lFingerB
- removed link lGripper
- added link L7, mass 2.3
Joints:
- removed joint LJFA
- removed joint LJFB
- joint LJFT: child lGripper -> L7

File: robots/alita/urdf/alita_right.urdf (robot description, URDF)
Before this commit: robot alita_right, 10 links, 9 joints
Links:
- removed link rFingerA
- removed link rFingerB
- removed link rGripper
- added link R7, mass 2.3
Joints:
- removed joint RJFA
- removed joint RJFB
- joint RJFT: child rGripper -> R7
