Commit message: Added models for general use of Alita as bimanual robot

File: robots/alita/urdf/alita_hand.urdf (robot description, URDF)
Before this commit: robot alita_left, 4 links, 3 joints
Links:
- removed link gripper
- added link alita_palm, mass 2.3; collision box size=0.15 0.125 0.210; visual mesh filename=../meshes/Schunk/SchunkGripper/L7.dae
Joints:
- joint LJFA: parent gripper -> alita_palm
- joint LJFB: parent gripper -> alita_palm
- joint LJFT: child gripper -> alita_palm

Commit message: Added left and right modification for alita arms

File: robots/alita/urdf/alita_hand.urdf (robot description, URDF)
Before this commit: robot alita_hand, 4 links, 3 joints
Joints:
- joint LJFA: limit lower=0.0 upper=0.030 effort=1000 velocity=0.1 -> lower=0.0 upper=0.070 effort=1000 velocity=0.1; origin xyz=-0.05 0.00 0.127 rpy=3.1416 0.0 0.0 -> xyz=0.0 0.00 0.127 rpy=3.1416 0.0 0.0
- joint LJFB: limit lower=0.0 upper=0.030 effort=1000 velocity=0.1 -> lower=0.0 upper=0.070 effort=1000 velocity=0.1; origin xyz=0.050 -0.00 0.127 rpy=0 3.1416 0.0 -> xyz=0.0 -0.00 0.127 rpy=0 3.1416 0.0

File: robots/alita/urdf/alita_left.urdf (robot description, URDF)
Before this commit: robot alita_left, 9 links, 8 joints
Joints:
- joint LJ1: limit lower=-4.7124 upper=4.7124 effort=1000 velocity=0.1 -> lower=-3.14157 upper=3.14157 effort=1000 velocity=0.1
- joint LJ2: limit lower=-2.094 upper=2.094 effort=1000 velocity=0.1 -> lower=-1.5708 upper=1.5708 effort=1000 velocity=0.1
- joint LJ3: limit lower=-4.7124 upper=4.7124 effort=1000 velocity=0.1 -> lower=-3.14157 upper=3.14157 effort=1000 velocity=0.1
- joint LJ4: limit lower=-2.094 upper=2.094 effort=1000 velocity=0.1 -> lower=-1.919 upper=1.919 effort=1000 velocity=0.1
- joint LJ5: limit lower=-4.7124 upper=4.7124 effort=1000 velocity=0.1 -> lower=-3.14157 upper=3.14157 effort=1000 velocity=0.1
- joint LJ6: limit lower=-2.094 upper=2.094 effort=1000 velocity=0.1 -> lower=-1.745 upper=1.745 effort=1000 velocity=0.1
- joint LJFT: limit lower=-4.7124 upper=4.7124 effort=1000 velocity=0.1 -> lower=-3.14157 upper=3.14157 effort=1000 velocity=0.1

File: robots/alita/urdf/alita_right.urdf (robot description, URDF)
Before this commit: robot alita_right, 8 links, 7 joints
Joints:
- joint RJ1: limit lower=-4.7124 upper=4.7124 effort=1000 velocity=0.1 -> lower=-3.14157 upper=3.14157 effort=1000 velocity=0.1
- joint RJ2: limit lower=-2.094 upper=2.094 effort=1000 velocity=0.1 -> lower=-1.5708 upper=1.5708 effort=1000 velocity=0.1
- joint RJ3: limit lower=-4.7124 upper=4.7124 effort=1000 velocity=0.1 -> lower=-3.14157 upper=3.14157 effort=1000 velocity=0.1
- joint RJ4: limit lower=-2.094 upper=2.094 effort=1000 velocity=0.1 -> lower=-1.919 upper=1.919 effort=1000 velocity=0.1
- joint RJ5: limit lower=-4.7124 upper=4.7124 effort=1000 velocity=0.1 -> lower=-3.14157 upper=3.14157 effort=1000 velocity=0.1
- joint RJ6: limit lower=-2.094 upper=2.094 effort=1000 velocity=0.1 -> lower=-1.745 upper=1.745 effort=1000 velocity=0.1
- joint RJFT: limit lower=-4.7124 upper=4.7124 effort=1000 velocity=0.1 -> lower=-3.14157 upper=3.14157 effort=1000 velocity=0.1

Commit message: Added correction in hand module

File: robots/alita/urdf/alita_hand.urdf (robot description, URDF)
Before this commit: robot alita_hand, 4 links, 3 joints
Links:
- link fingerA: geometry collision mesh filename=../meshes/Schunk/SchunkGripper/gripperPlate.dae; visual mesh filename=../meshes/Schunk/SchunkGripper/gripperPlate.dae
- link fingerB: geometry collision mesh filename=../meshes/Schunk/SchunkGripper/gripperPlate.dae; visual mesh filename=../meshes/Schunk/SchunkGripper/gripperPlate.dae

Commit message: Updated hand module according to real hand

File: robots/alita/urdf/alita_hand.urdf (robot description, URDF)
Before this commit: robot alita_hand, 4 links, 3 joints
Joints:
- joint LJFA: axis 1 0 0 -> -1 0 0; limit lower=0.0 upper=0.070 effort=1000 velocity=0.1 -> lower=0.0 upper=0.035 effort=1000 velocity=0.1; origin xyz=0.0 0.00 0.127 rpy=3.1416 0.0 0.0 -> xyz=0.02 0.00 0.127 rpy=0.0 3.1416 0.0
- joint LJFB: axis 1 0 0 -> -1 0 0; limit lower=0.0 upper=0.070 effort=1000 velocity=0.1 -> lower=0.0 upper=0.035 effort=1000 velocity=0.1; origin xyz=0.0 -0.00 0.127 rpy=0 3.1416 0.0 -> xyz=-0.02 0.00 0.127 rpy=3.1416 0.0 0.0

Commit message: Added fullpath for testing

File: robots/alita/urdf/alita_hand.urdf (robot description, URDF)
Before this commit: robot alita_hand, 4 links, 3 joints
Joints:
- joint LJFA: origin xyz=0.02 0.00 0.127 rpy=0.0 3.1416 0.0 -> xyz=0.035 0.00 0.127 rpy=0.0 3.1416 0.0
- joint LJFB: origin xyz=-0.02 0.00 0.127 rpy=3.1416 0.0 0.0 -> xyz=-0.035 0.00 0.127 rpy=3.1416 0.0 0.0

File: robots/lwa4d/urdf/lwa4d_right_phys_box.urdf (robot description, URDF)
Before this commit: robot lwa4d_right, 9 links, 8 joints
Links:
- link L1_link: geometry collision mesh filename=../meshes/arm_1_link_box_12.dae; visual mesh filename=../meshes/arm_1_link.dae
- link L2_link: geometry collision mesh filename=../meshes/arm_2_link_box_12.dae; visual mesh filename=../meshes/arm_2_link.dae
- link L4_link: geometry collision mesh filename=../meshes/arm_4_link_box_12.dae; visual mesh filename=../meshes/arm_4_link.dae
- link L5_link: geometry collision mesh filename=../meshes/arm_5_link_phys_box_12.dae; visual mesh filename=../meshes/arm_5_link_phys.dae
- link L6_link: geometry collision mesh filename=../meshes/arm_6_link_box_12.dae; visual mesh filename=../meshes/arm_6_link.dae
- link L7_link: geometry collision mesh filename=../meshes/arm_7_FT_tool_changers_link_box_12.dae; visual mesh filename=../meshes/arm_7_FT_tool_changers_link.dae
Joints:
- joint L1_joint: limit lower=-3.14157 upper=3.14157 effort=370 velocity=2.0 -> lower=-2.91 upper=2.91 effort=370 velocity=2.0
- joint L2_joint: limit lower=-1.97 upper=1.97 effort=370 velocity=2.0 -> lower=-1.92 upper=1.92 effort=370 velocity=2.0
- joint L3_joint: limit lower=-3.14157 upper=3.14157 effort=176 velocity=2.0 -> lower=-2.91 upper=2.91 effort=176 velocity=2.0
- joint L4_joint: limit lower=-2.08208 upper=2.08208 effort=176 velocity=2.0 -> lower=-1.95 upper=1.95 effort=176 velocity=2.0
- joint L5_joint: limit lower=-3.14157 upper=3.14157 effort=41.6 velocity=2.0 -> lower=-2.91 upper=2.91 effort=41.6 velocity=2.0
- joint L6_joint: limit lower=-1.8 upper=1.8 effort=20.1 velocity=2.0 -> lower=-1.78 upper=1.78 effort=20.1 velocity=2.0
- joint L7_joint: limit lower=-3.14157 upper=3.14157 effort=9.6 velocity=2.0 -> lower=-2.74 upper=2.74 effort=9.6 velocity=2.0
