Commit message: Added last changes

File: objects/basicShapes/urdf/ball_01.urdf (robot description, URDF)
Before this commit: robot ball_01, 1 links, 0 joints
Links:
- link ball_01: geometry visual sphere radius=0.01

File: robots/alita/urdf/alita_hand.urdf (robot description, URDF)
Before this commit: robot alita_hand, 4 links, 3 joints
Links:
- link fingerA: geometry collision mesh filename=../meshes/alita-finger.dae; visual mesh filename=../meshes/alita-finger.dae
- link fingerB: geometry collision mesh filename=../meshes/alita-finger.dae; visual mesh filename=../meshes/alita-finger.dae
