Commit message: Modified palm mesh in sdh to have fingers aligned with X axis

File: robots/sdh/urdf/sdh_original.urdf (robot description, URDF)
Before this commit: robot sdh, 13 links, 12 joints
Joints:
- joint finger_21_joint: origin xyz=-0.033 -0.01905 0.0745 rpy=0 0 1.5708 -> xyz=0.01905 -0.033 0.0745 rpy=0 0 3.14159265
- joint knuckle_joint: origin xyz=0.033 -0.01905 0.0745 rpy=0 0 1.5708 -> xyz=0.01905 0.033 0.0745 rpy=0 0 3.14159265
- joint thumb_1_joint: origin xyz=0 0.03811 0.0745  rpy=0 0 -1.5708 -> xyz=-0.03811 0 0.0745  rpy=0 0 0
