Commit message: Added changes of Wednesday

File: robots/sdh/urdf/sdh.urdf (robot description, URDF)
Before this commit: robot sdh, 13 links, 12 joints
Links:
- link finger_12_link: geometry collision mesh filename=../meshes/finger_niceMesh.dae; visual mesh filename=../meshes/finger_niceMesh.dae
- link finger_22_link: geometry collision mesh filename=../meshes/finger_niceMesh.dae; visual mesh filename=../meshes/finger_niceMesh.dae
- link thumb_2_link: geometry collision mesh filename=../meshes/finger_niceMesh.dae; visual mesh filename=../meshes/finger_niceMesh.dae
