Commit message: Added box-like crichton

File: objects/kiva_pod/urdf/kiva_pod.urdf (robot description, URDF)
Before this commit: robot kiva_pod, 1 links, 0 joints
Links:
- link kiva_pod: geometry collision mesh filename=../meshes/mesh_adapted_golems.dae scale=1 1 1; visual mesh filename=../meshes/mesh_adapted_golems.dae scale=1 1 1
