Commit message: Added gripper models

File: robots/baxter/urdf/baxter_left_arm.urdf (robot description, URDF)
Before this commit: robot baxter_left_arm, 13 links, 12 joints
Links:
- removed link left_upper_elbow_visual
- removed link left_upper_forearm_visual
- removed link torso
- added link left_arm_root
- link left_upper_elbow: geometry collision cylinder length=0.107 radius=0.06; collision cylinder length=0.273 radius=0.06
- link left_upper_forearm: geometry collision cylinder length=0.088 radius=0.06; collision cylinder length=0.272 radius=0.06
Joints:
- removed joint left_e0_fixed
- removed joint left_torso_arm_mount
- removed joint left_w0_fixed
- removed joint torso_t0
- added joint left_arm_root_joint: type floating, parent world, child left_arm_root, origin xyz=0 0 0 rpy=0 0 0
- added joint left_arm_root_mount: type fixed, parent left_arm_root, child left_arm_mount, origin xyz=0.024645 0.219645 0.118588 rpy=0 0 0.7854

File: robots/baxter/urdf/baxter_right_arm.urdf (robot description, URDF)
Before this commit: robot baxter_right_arm, 13 links, 12 joints
Links:
- removed link right_upper_elbow_visual
- removed link right_upper_forearm_visual
- removed link torso
- added link right_arm_root
- link right_upper_elbow: geometry collision cylinder length=0.107 radius=0.06; collision cylinder length=0.273 radius=0.06
- link right_upper_forearm: geometry collision cylinder length=0.088 radius=0.06; collision cylinder length=0.272 radius=0.06
Joints:
- removed joint right_e0_fixed
- removed joint right_w0_fixed
- removed joint torso_t0
- added joint right_arm_root_joint: type floating, parent world, child right_arm_root, origin xyz=0 0 0 rpy=0 0 0
- joint right_torso_arm_mount: parent torso -> right_arm_root

File: robots/baxter/urdf/baxter_torso.urdf (robot description, URDF)
Before this commit: robot baxter, 10 links, 9 joints
Links:
- removed link left_torso_itb
- removed link right_torso_itb
- link screen: geometry collision sphere radius=0.001; visual mesh filename=/home/ana/Research/commonData/robots/baxter/meshes/head/H1_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
Joints:
- removed joint left_torso_itb_fixed
- removed joint right_torso_itb_fixed
