Commit message: Trying to fix the FCL issue

File: objects/utils/urdf/yellow_cylinder.urdf (robot description, URDF)
Before this commit: robot yellow_cylinder, 1 links, 0 joints
Links:
- link yellow_cylinder: geometry collision mesh filename=../meshes/yellow_cylinder_010_024_s8.dae scale=1 1 1; visual mesh filename=../meshes/yellow_cylinder_010_024_s8.dae scale=1 1 1

Commit message: Added meshes experiments to get collision good

File: objects/utils/urdf/yellow_cylinder.urdf (robot description, URDF)
Before this commit: robot yellow_cylinder, 1 links, 0 joints
Links:
- link yellow_cylinder: geometry collision mesh filename=../meshes/yellow_cylinder_010_024.dae scale=1 1 1; visual mesh filename=../meshes/yellow_cylinder_010_024.dae scale=1 1 1
