Commit message: Added meshes

File: objects/utils/urdf/red_cup_8_9_9.urdf (robot description, URDF)
Before this commit: robot sq_cylinder_10_20, 1 links, 0 joints
Links:
- removed link sq_cylinder_10_20
- added link red_cup_8_9_(, mass 0.5; collision mesh filename=../meshes/red_cup_8_9_9.dae scale=1 1 1; visual mesh filename=../meshes/red_cup_8_9_9.dae scale=1 1 1

Commit message: Corrected name on cup

File: objects/utils/urdf/red_cup_8_9_9.urdf (robot description, URDF)
Before this commit: robot red_cup_8_9_9, 1 links, 0 joints
Links:
- removed link red_cup_8_9_(
- added link red_cup_8_9_9, mass 0.5; collision mesh filename=../meshes/red_cup_8_9_9.dae scale=1 1 1; visual mesh filename=../meshes/red_cup_8_9_9.dae scale=1 1 1
