Commit message: Added alita scenarios for marker and skeleton tracker test

File: objects/shelf_RIM/urdf/shelf_RIM.urdf (robot description, URDF)
Before this commit: robot shelf_RIM, 1 links, 0 joints
Links:
- link shelf_RIM: geometry collision mesh filename=../meshes/paddedShelf.dae scale=1 1 1; visual mesh filename=../meshes/lab_shelf.stl scale=1 1 1

Commit message: Added 9 objects for ch3

File: objects/shelf_RIM/urdf/shelf_RIM.urdf (robot description, URDF)
Before this commit: robot shelf_RIM, 1 links, 0 joints
Links:
- link shelf_RIM: geometry collision mesh filename=../meshes/shelf_RIM.dae scale=1 1 1; visual mesh filename=../meshes/shelf_RIM.dae scale=1 1 1
